Commit message: Update ur10e_robot.urdf.xacro

File: robot/ur10e_robot.urdf.xacro (robot description, xacro)
@@ -21,5 +21,6 @@
     <parent link="tool0" />
     <child link = "hand" />
-    <origin xyz="0 -0.135 0.04" rpy="1.5758 3.1415 1.5758" />
+  <!--  <origin xyz="0 -0.135 0.04" rpy="1.5758 3.1415 1.5758" /> -->
+         <origin xyz="0 0 0.1" rpy="0 0 0" />
   </joint>
 </robot>

Commit message: Update ur10e_robot.urdf.xacro

File: robot/ur10e_robot.urdf.xacro (robot description, xacro)
@@ -21,6 +21,5 @@
     <parent link="tool0" />
     <child link = "hand" />
-  <!--  <origin xyz="0 -0.135 0.04" rpy="1.5758 3.1415 1.5758" /> -->
-         <origin xyz="0 0 0.1" rpy="0 0 0" />
+  <origin xyz="0 -0.135 0.04" rpy="1.5758 3.1415 1.5758" />
   </joint>
 </robot>
